File: ch32v203-promicro/ch32v203-promicro.kicad_pcb (KiCad board)
At the start: 2 copper layers, 17.8 x 33 mm, 28 parts, among them J1 USB2.0_C_v3, J2 ProMicro-LeftPin, J3 ProMicro-RightPin, SW1 SW_Push, SW2 SW_Push, U1 CH32V203CxT6, U2 AMS1117-3.3, Y1 32.768k, Y2 Crystal_GND24

Commit message: ch32v203micro
Parts:
- removed REF**: JLCJLCJLCJLC, $74th:JLCJLCJLCJLC
- Y1: footprint Crystal:Crystal_SMD_3215-2Pin_3.2x1.5mm -> $74th:Crystal_SMD_3215-2Pin_3.2x1.5mm
- Y2: value Crystal_GND24 -> 8M
Routing:
- net Net-(R6-Pad1): track 4.89 -> 6.64 mm
- net GND: track 79.3 -> 78.0 mm
- net RST: track 31.3 -> 32.0 mm
- net DP: track 28.4 -> 27.7 mm
- net 6/A7: track 12.0 -> 11.4 mm

Commit message: ch32v203micro v1.0.0
Parts:
- turned R2 to 0 degrees
Connections:
- C6 pad 1: Net-(C6-Pad1) -> RST
- R2 pad 1: Net-(C6-Pad1) -> +3V3
- R2 pad 2: GND -> RST
- R6 pad 1: Net-(R6-Pad1) -> Net-(U1-Pad44)
- R7 pad 1: +3V3 -> Net-(U1-Pad20)
- R7 pad 2: Net-(R7-Pad2) -> GND
- SW1 pad 1: Net-(C6-Pad1) -> GND
- SW2 pad 1: Net-(R7-Pad2) -> Net-(U1-Pad44)
- SW2 pad 2: Net-(SW2-Pad2) -> +3V3
- U1 pad 20: Net-(SW2-Pad2) -> Net-(U1-Pad20)
- U1 pad 32: unconnected-(U1-Pad32) -> DM
- U1 pad 33: unconnected-(U1-Pad33) -> DP
- U1 pad 42: DM -> unconnected-(U1-Pad42)
- U1 pad 43: DP -> unconnected-(U1-Pad43)
- U1 pad 44: Net-(R6-Pad1) -> Net-(U1-Pad44)
Routing:
- net GND: track 78.0 -> 98.7 mm, vias 23 -> 25
- net Net-(SW2-Pad2): track 19.3 -> 0.00 mm, vias 2 -> 0
- net Net-(U1-Pad44): track 0.00 -> 15.5 mm, vias 0 -> 1
- net +3V3: track 50.4 -> 64.4 mm
- net Net-(U1-Pad20): track 0.00 -> 10.5 mm, vias 0 -> 1
- net Net-(C6-Pad1): track 9.47 -> 0.00 mm, vias 2 -> 0
- net Net-(R7-Pad2): track 9.08 -> 0.00 mm, vias 1 -> 0
- net Net-(R6-Pad1): track 6.64 -> 0.00 mm, vias 1 -> 0
- net RST: track 32.0 -> 36.6 mm
- net 6/A7: track 11.4 -> 8.85 mm
- net DP: track 27.7 -> 25.5 mm, vias 4 -> 2
- net 10/A10: track 26.8 -> 25.2 mm
- net DM: track 29.9 -> 28.5 mm, vias 4 -> 2
- net Net-(R3-Pad2): track 3.29 -> 4.69 mm
- net 4/A6: track 4.76 -> 3.95 mm
