File: ch32v203-promicro/ch32v203-promicro.kicad_sch (KiCad schematic)
At the start: 29 parts, among them J1 USB2.0_C_v3, J2 ProMicro-LeftPin-NoGND, J3 ProMicro-RightPin, SW1 SW_Push, SW2 SW_Push, U1 STM32V103C8T6, U2 AMS1117-3.3, Y1 32.768k, Y2 8M

Commit message: v1.2.0
Parts:
- removed C8: 12p, $74th:Capacitor_0805_2012, symbol Device:C
- removed J2: ProMicro-LeftPin-NoGND, $74th:ProMicro_LIKE_LEFT_NO_GND, symbol $74th:ProMicro-LeftPin-NoGND
- removed J3: ProMicro-RightPin, $74th:ProMicro_LIKE_RIGHT, symbol $74th:ProMicro-RightPin
- removed JP1: Jumper_3_Open, Jumper:SolderJumper-3_P1.3mm_Open_RoundedPad1.0x1.5mm, symbol Jumper:Jumper_3_Open
- removed R3: 0, $74th:Register_0805_2012, symbol Device:R
- removed R6: 10k, $74th:Register_0805_2012, symbol Device:R
- removed Y1: 32.768k, $74th:Crystal_SMD_3215-2Pin_3.2x1.5mm, symbol Device:Crystal
- added C11: 1u, $74th:Capacitor_0805_2012, symbol Device:C
- added J5: ProMicro-LeftPin-NoGND, $74th:ProMicro_LIKE_LEFT_NO_GND, symbol $74th:ProMicro-LeftPin-NoGND
- added J6: ProMicro-RightPin, $74th:ProMicro_LIKE_RIGHT, symbol $74th:ProMicro-RightPin
- added R9: 27.4, $74th:Register_0805_2012, symbol Device:R
- added U4: CH213K, Package_TO_SOT_SMD:SOT-23, symbol $74th:CH213K-Ideal_Diode_for_USB_Power
- C5: value 2.2u -> 10u
- C7: value 12p -> 100n
- D1: value LED -> BLUE
- R1: value 200 -> 10k
- R2: value 10k -> 27.4
- U1: value STM32V103C8T6 -> CH32V203C8T6
Connections:
- net +3V3: now also C7.1, SW2.1, U1.1 (VBAT), U1.9 (VDDA), C11.1, J6.9 (3V3); no longer R2.1, SW1.1
- net +5V: now also J6.12 (RAW), U4.3 (VI+); no longer C4.1, U2.3 (VI)
- net 0/UART_RX: now also J5.2 (0/RX)
- net 10/A10: now also J6.1 (10/A10)
- net 14/SPI_MISO: now also J6.3 (14/SPI_MISO)
- net 15/SPI_SCK: now also J6.4 (15/SPI_SCK)
- net 16/SPI_MOSI: now also J6.2 (16/SPI_MOSI)
- net 18/A0: now also J6.5 (18/A0)
- net 19/A1: now also J6.6 (19/A1)
- net 1/UART_TX: now also J5.1 (1/TX)
- net 20/A2: now also J6.7 (20/A2)
- net 21/A3: now also J6.8 (21/A3)
- net 4/A6: now also U1.19 (PB1/ADC9), J5.7 (4/A6); no longer U1.40 (PB4/JNTRST)
- net 5: now also U1.39 (PB3/JTDO), J5.8 (5); no longer U1.18 (PB0/ADC8)
- net 6/A7: now also U1.18 (PB0/ADC8), J5.9 (6/A7); no longer U1.39 (PB3/JTDO)
- net 7: now also U1.40 (PB4/JNTRST), J5.10 (7); no longer U1.19 (PB1/ADC9)
- net 8/A8: now also J5.11 (8/A8)
- net 9/A9: now also J5.12 (9/A9)
- net GND: now also SW1.2, C11.2, J6.11 (GND), U4.1 (GND)
- net SWCLK: now also J5.4 (Alt2)
- net SWDIO: now also J5.3 (Alt1)
- net at U1.3 (PC14/OSC32IN): no longer C7.1
- net 2/I2C_SDA renamed 2/ISC_SDA
- net 2/ISC_SDA: now also J5.5 (2/SDA)
- net 3/I2C_SCL renamed 3/ISC_SCL
- net 3/ISC_SCL: now also J5.6 (3/SCL)
- net BOOT0: no longer names the net of R8.1, SW2.2, U1.44 (BOOT0)
- net BOOT0: no longer C6.1, R2.2
- net BOOT1: no longer names the net of R7.1, U1.20 (BOOT1/PB2)
- net DM: no longer names the net of J1.2 (D-)
- net DM: now also R2.1; no longer U1.32 (PA11/UART1_CTS/USBDM)
- net DP: no longer names the net of J1.3 (D+)
- net DP: now also R9.1; no longer U1.33 (PA12/UART1_RTS/USBDP)
- net RST renamed ~{RESET}
- net ~{RESET}: now also C6.1, SW1.1, J6.10 (~{RESET}); no longer SW1.2
- new net: C4.1, U2.3 (VI), U4.2 (VO-)
- new net USB_DM: R2.2, U1.32 (PA11/UART1_CTS/USBDM)
- new net USB_DP: R9.2, U1.33 (PA12/UART1_RTS/USBDP)
- no-connect marks 11 -> 12
Other:
- note added: "MCU"
- note added: "Power"
- note added: "ProMicro"
- note added: "USB"
- company: (none) -> 74th
- title: STM32Micro -> CH32V203Micro
- moved on the sheet: C1, C10, C2, C3, C4, C5, C6, D1, J1, R1, R4, R5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

Commit message: ch32v203 promicro v1.2.1
Parts:
- renumbered C4 to C1, C5 to C2, C11 to C3, C7 to C4, C1 to C5, C3 to C6, C2 to C7, C6 to C8, J5 to J2, J6 to J3, R5 to R1, R4 to R2, R1 to R3, R2 to R4, R9 to R5, R7 to R6, R8 to R7, SW2 to SW1, SW1 to SW2, U2 to U1, U1 to U2, U4 to U3, Y2 to Y1

Commit message: update kicad version
Parts:
- C1, C10, C2, C3, C4, C5, C6, C7, C8, C9: footprint $74th:Capacitor_0805_2012 -> 74th:Capacitor_0805_2012
- D1: footprint $74th:LED_0805_2012Metric_Pad1.15x1.40mm_HandSolder -> 74th:LED_0805_2012
- J1: footprint $74th:USB-C-12-Pin-SMD -> 74th:Connector_USB-C-Receptacle_SMT_12-Pin_Simple; symbol $74th:USB2.0_C_v3 -> 74th_Interface:USB_TypeC-2.0_Receptacle_Simple
- J2: footprint $74th:ProMicro_LIKE_LEFT_NO_GND -> 74th:PinOut_ProMicro-LIKE_LEFT_NO-GND; symbol $74th:ProMicro-LeftPin-NoGND -> 74th_Interface:ProMicro-Left_NoGND
- J3: footprint $74th:ProMicro_LIKE_RIGHT -> 74th:PinOut_ProMicro-LIKE_RIGHT; symbol $74th:ProMicro-RightPin -> 74th_Interface:ProMicro-Right
- R1, R2, R3, R4, R5, R6, R7: footprint $74th:Register_0805_2012 -> 74th:Register_0805_2012
- SW1, SW2: footprint $74th:SKRPABE010 -> 74th:Switch_SKRPABE010
- U1: footprint Package_TO_SOT_SMD:SOT-89-3_Handsoldering -> 74th:Package_SOT-89-3
- U2: footprint Package_QFP:LQFP-48_7x7mm_P0.5mm -> 74th:Package_LQFP-48_7x7mm_P0.5mm; symbol $74th:STM32F103C8T6 -> 74th_MCU:CH32V203CxT6
- U3: footprint Package_TO_SOT_SMD:SOT-23 -> 74th:Package_SOT-23; symbol $74th:CH213K-Ideal_Diode_for_USB_Power -> 74th_Passive:CH213K_Ideal-Diode-for-USB-Power
- Y1: footprint $74th:Crystal_SMD_3225-4Pin_3.2x2.5mm_HandSoldering -> 74th:Crystal_SMD_3225-4Pin_3.2x2.5mm_HandSoldering
