File: ch32x035-promicro-usb-pd/ch32x035-promicro-usb-pd.kicad_sch (KiCad schematic)
At the start: 33 parts, among them J1 USB_TypeC-2.0_Receptacle, SW1 SW_Push, U1 CH32X035G8U6, U3 TPS562203, U4 AMS1117-3.3(NC)

Commit message: ch32x035-usb-device
Parts:
- removed F1: Polyfuse, symbol Device:Polyfuse
- removed R12, R13: 1k(NC), symbol Device:R
- C1, C10, C2, C3, C4, C5, C6, C7, C8, C9: footprint (none) -> 74th:Capacitor_0603_1608
- CH1: footprint (none) -> 74th:ProMicro-LIKE_RIGHT
- CH2: footprint (none) -> 74th:ProMicro-LIKE_LEFT_NO-GND
- J1: footprint (none) -> 74th:USB-C-Receptacle_SMD_12-Pin
- JP1: footprint (none) -> Jumper:SolderJumper-2_P1.3mm_Open_RoundedPad1.0x1.5mm
- L1, R1, R10, R11, R2, R3, R4, R5, R6, R7, R8, R9: footprint (none) -> 74th:Register_0603_1608
- SW1: footprint (none) -> 74th:PushButton_SKRPABE010
- U1: footprint Package_DFN_QFN:QFN-28-1EP_4x4mm_P0.4mm_EP2.3x2.3mm -> 74th:QFN-28-1EP_4x4mm_P0.4mm_EP2.8x2.8mm_hand-solder
- U3: footprint (none) -> Package_TO_SOT_SMD:SOT-23-6_Handsoldering
Connections:
- net VBUS: now also J1.1 (VBUS); no longer R9.2
- net VDD: now also R9.2
- net ~{RESET}: now also U3.5 (EN); no longer U3.7 (EN)
Other:
- note added: "PD Power Step Down"
- note removed: "PD Power"
- company: (none) -> @74th
- title: (none) -> ch32x035 ProMicro
- moved on the sheet: R1, R2, R9

Commit message: v1.2.0
Parts:
- removed C2: 10u, 74th:Capacitor_0603_1608, symbol Device:C
- removed C3: 100n, 74th:Capacitor_0603_1608, symbol Device:C
- removed C7: NC, 74th:Capacitor_0603_1608, symbol Device:C
- removed JP1: Jumper_2_Open, Jumper:SolderJumper-2_P1.3mm_Open_RoundedPad1.0x1.5mm, symbol Jumper:Jumper_2_Open
- removed R1, R2: 27, 74th:Register_0603_1608, symbol Device:R
- removed R10, R11, R8: 0(NC), 74th:Register_0603_1608, symbol Device:R
- removed R3, R4: 5.1k, 74th:Register_0603_1608, symbol Device:R
- removed R9: 1.5k, 74th:Register_0603_1608, symbol Device:R
- removed U4: AMS1117-3.3(NC), Package_TO_SOT_SMD:SOT-89-3, symbol 74th_Passive:AMS1117-3.3_Regulator_SOT89
- added CH3: 3Pin, 74th:PinOut_3Pin, symbol 74th_Interface:3Pin
- added CH4: 2Pin, 74th:PinOut_2Pin, symbol 74th_Interface:2Pin
- C1: value 10u -> 22u; footprint 74th:Capacitor_0603_1608 -> 74th:Capacitor_0805_2012
- C10, C4, C5, C6, C8, C9: footprint 74th:Capacitor_0603_1608 -> 74th:Capacitor_0805_2012
- CH1: footprint 74th:ProMicro-LIKE_RIGHT -> 74th:PinOut_ProMicro-LIKE_RIGHT
- CH2: footprint 74th:ProMicro-LIKE_LEFT_NO-GND -> 74th:PinOut_ProMicro-LIKE_LEFT_NO-GND
- J1: footprint 74th:USB-C-Receptacle_SMD_12-Pin -> 74th:Connector_USB-C-Receptacle_SMT_12-Pin_Simple
- L1, R5: footprint 74th:Register_0603_1608 -> 74th:Register_0805_2012
- R6: value 135k -> 100k; footprint 74th:Register_0603_1608 -> 74th:Register_0805_2012
- R7: value 30k -> 22k; footprint 74th:Register_0603_1608 -> 74th:Register_0805_2012
- U1: footprint 74th:QFN-28-1EP_4x4mm_P0.4mm_EP2.8x2.8mm_hand-solder -> 74th:Package_QFN-28-1EP_4x4mm_P0.4mm_EP2.8x2.8mm
- U3: value TPS562203 -> MT2492; footprint Package_TO_SOT_SMD:SOT-23-6_Handsoldering -> 74th:Package_SOT-23-6; symbol 74th_Passive:TPS56220x_Step-Down-DCDC-Converter -> 74th_Passive:MT2492_Step-Down-DCDC-Converter
Connections:
- net USB_DM is gone; now on net 20/A2: U1.26 (PC16/UDM)
- net USB_DP is gone; now on net 21/A3: U1.27 (PC17/UDP)
- net 10/A10: now also U1.14 (PB3/TX3/C3O/O2P1); no longer U1.9 (PA4/CS/CK2/O2O0/A4)
- net 14/SPI_MISO: now also U1.18 (PB7/T1C2N/O2P2/RTS3); no longer U1.11 (PA6/MISO/T3C1/O1N0/A6)
- net 15/SPI_SCK: now also U1.19 (PB8/T1C3N/O1P1); no longer U1.10 (PA5/SCK/O2N0/A5)
- net 16/SPI_MOSI: now also U1.16 (PB1/RX4/O2N1/A9/PB5/CK3/O1O1/T1BK); no longer U1.12 (PA7/MOSI/T3C2/O2P0/A7)
- net 18/A0: now also U1.20 (PB9/CK1/T1C1/MCO); no longer U1.5 (PA0/T2C1/CTS2/C1P1/A0)
- net 19/A1: now also U1.23 (PB12); no longer U1.6 (PA1/RTS2/T2C2/C10/O1N2/O2N2/A1)
- net 20/A2: no longer U1.7 (PA2/TX2/T2C3/O2O1/C3N0/A2)
- net 21/A3: no longer U1.8 (PA3/RX2/T2C4/O1O0/A3)
- net 2/SDA: now also U1.3 (PC0/A10); no longer U1.13 (PB0/TX4/O1P0/A8)
- net 3/SCL: now also U1.4 (PC3/C1N0/C2N1/C3N1/A13); no longer U1.16 (PB1/RX4/O2N1/A9/PB5/CK3/O1O1/T1BK)
- net 4/A6: now also U1.5 (PA0/T2C1/CTS2/C1P1/A0); no longer U1.14 (PB3/TX3/C3O/O2P1)
- net 5: now also U1.6 (PA1/RTS2/T2C2/C10/O1N2/O2N2/A1); no longer U1.15 (PB4/RX3/O1P2)
- net 6/A7: now also U1.7 (PA2/TX2/T2C3/O2O1/C3N0/A2); no longer U1.17 (PB6/T1C1N/CTS3/O1N1)
- net 7: now also U1.8 (PA3/RX2/T2C4/O1O0/A3); no longer U1.23 (PB12)
- net 8/A8: now also U1.10 (PA5/SCK/O2N0/A5); no longer U1.19 (PB8/T1C3N/O1P1)
- net 9/A9: now also U1.12 (PA7/MOSI/T3C2/O2P0/A7); no longer U1.20 (PB9/CK1/T1C1/MCO)
- net GND: now also U3.2 (GND); no longer U3.1 (GND)
- net VBUS: now also U3.5 (VIN); no longer U3.3 (VIN)
- net VDD: now also R6.2; no longer R6.1
- net at C6.1, L1.1: now also U3.6 (SW); no longer U3.2 (SW)
- net at C6.2: now also U3.1 (BS); no longer U3.4 (BST)
- net ~{RESET} renamed RESET
- net RESET: now also U3.4 (EN); no longer U3.5 (EN)
- new net DCDC-FB: R6.1, R7.1, U3.3 (FB)
- new net G0: CH3.1, U1.9 (PA4/CS/CK2/O2O0/A4)
- new net G1: CH3.2, U1.11 (PA6/MISO/T3C1/O1N0/A6)
- new net G2: CH3.3, U1.13 (PB0/TX4/O1P0/A8)
- new net G3: CH4.1, U1.17 (PB6/T1C1N/CTS3/O1N1)
- new net G4: CH4.2, U1.15 (PB4/RX3/O1P2)
Other:
- note removed: "Direct USB 5V Power(Alternate)"
- note removed: "Non PD Power(Alternate)"
- note removed: "PC16,17をI2Cで使う場合や、USB DM/DPを使わない場合、 R1-2,9をNCにする"
- note removed: "PC16,17をI2Cとして使う場合、R8,10,12-13を実装する"
- note removed: "PDを使い場合のみ。 PDを使わない場合でも、C1-2,5-6 は必要。"
- note removed: "PDを使う場合はR11をNCにする その時はDCDC ConverterのENがリセットとして機能する"
- note removed: "PDを使う場合はR3、R4をNCにする"
- note removed: "USB 5VからVDD=3.3Vにする場合のみ"
- note removed: "USB 5VからVDD=5Vにする場合のみ、ジャンパさせる"
- moved on the sheet: C1, C4, C5, C6, CH1, CH2, J1, L1, R5, R6, R7, U3

Commit message: ch32x035
Parts:
- U1: footprint 74th:Package_QFN-28-1EP_4x4mm_P0.4mm_EP2.8x2.8mm -> 74th:QFN-28-1EP_4x4mm_P0.4mm_EP2.8x2.8mm
Changed lines of the file:
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@@
       (effects (font (size 1.27 1.27)) (justify left))
     )
-    (property "Footprint" "74th:Package_QFN-28-1EP_4x4mm_P0.4mm_EP2.8x2.8mm" (at 81.28 29.21 0)
+    (property "Footprint" "74th:QFN-28-1EP_4x4mm_P0.4mm_EP2.8x2.8mm" (at 81.28 29.21 0)
       (effects (font (size 1.27 1.27)) hide)
     )

Commit message: ch32x035-usb-pd
Parts:
- removed C4: 22u, 74th:Capacitor_0805_2012, symbol Device:C
- removed C6, C8: 100n, 74th:Capacitor_0805_2012, symbol Device:C
- removed CH4: 2Pin, 74th:PinOut_2Pin, symbol 74th_Interface:2Pin
- removed L1: 4.7u, 74th:Register_0805_2012, symbol Device:L
- removed R6: 100k, 74th:Register_0805_2012, symbol Device:R
- removed R7: 22k, 74th:Register_0805_2012, symbol Device:R
- removed SW1: SW_Push, 74th:PushButton_SKRPABE010, symbol Switch:SW_Push
- removed U3: MT2492, 74th:Package_SOT-23-6, symbol 74th_Passive:MT2492_Step-Down-DCDC-Converter
- added D1: BLUE, 74th:LED_0805_2012, symbol Device:LED
- added R1, R2: 5.1k, 74th:Register_0805_2012, symbol Device:R
- added R3, R4: 27, 74th:Register_0805_2012, symbol Device:R
- added U2: AMS1117, Package_TO_SOT_SMD:SOT-89-3, symbol 74th_Passive:AMS1117-3.3_Regulator_SOT89
- added U3: CH213K, Package_TO_SOT_SMD:SOT-23, symbol $74th:CH213K-Ideal_Diode_for_USB_Power
- C1, C5: value 22u -> 10u
- R5: value 100k -> 10k
- U1: footprint 74th:QFN-28-1EP_4x4mm_P0.4mm_EP2.8x2.8mm -> 74th:Package_QFN-28-1EP_4x4mm_P0.4mm_EP2.8x2.8mm
Connections:
- net G3 is gone; now on net 20/A2: U1.17 (PB6/T1C1N/CTS3/O1N1)
- net G4 is gone; now on net 21/A3: U1.15 (PB4/RX3/O1P2)
- net RESET is gone; now on net GND: CH1.10 (~{RESET}), R5.2
- net 20/A2: no longer U1.26 (PC16/UDM)
- net 21/A3: no longer U1.27 (PC17/UDP)
- net GND: now also R1.2, R2.2, U2.1 (GND), U3.1 (GND)
- net SWCLK: now also U1.24 (PC19/SWCLK); no longer U1.25 (PC18/SWDIO)
- net SWDIO: now also U1.25 (PC18/SWDIO); no longer U1.24 (PC19/SWCLK)
- net USB_CC1: now also R1.1
- net USB_CC2: now also R2.1
- net VBUS: now also U2.3 (VI); no longer R5.1
- net VDD: now also D1.2 (A), U3.2 (VO-); no longer CH1.9 (3V3)
- net at J1.2 (D-): now also R3.2
- net at J1.3 (D+): now also R4.2
- new net: D1.1 (K), R5.1
- new net +3.3V: CH1.9 (3V3), U2.2 (VO), U3.3 (VI+)
- new net USB_DM: R3.1, U1.26 (PC16/UDM)
- new net USB_DP: R4.1, U1.27 (PC17/UDP)
- no-connect marks 2 -> 0
Other:
- note added: "Power"
- note removed: "PD Power Step Down"
- note removed: "RESET"
- moved on the sheet: C1, C5
