File: wchlinke-swd-adapter/wchlinke-swd-adapter.kicad_sch (KiCad schematic)
At the start: 2 parts, among them J1 SWD_10Pin_Debugger-Side, U1 SWD_WCH-LinkE_Header

Commit message: update README
Other:
- title: (none) -> WCH-LinkE SWD Adapter
Changed lines of the file:
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@@
 (kicad_sch (version 20230121) (generator eeschema)
   (paper "A4")
+  (title_block
+    (title "WCH-LinkE SWD Adapter")
+    (rev "v1.0.0")
+  )
   (junction (at 40.64 91.44) (diameter 0) (color 0 0 0 0)
   )
