File: rvswdio-programer/rvswdio-programer.kicad_sch (KiCad schematic)
At the start: 21 parts, among them J1 USB2.0-C_SMT, U1 CH32V003F4P6, U2 AMS1117, U3 CH217K

Commit message: it works
Parts:
- R6, R7, R8: value 10 -> 0
Changed lines of the file:
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@@
 			)
 		)
-		(property "Value" "10"
+		(property "Value" "0"
 			(at 100.33 85.09 90)
 			(effects
@@
 			)
 		)
-		(property "Value" "10"
+		(property "Value" "0"
 			(at 100.33 68.58 90)
 			(effects
@@
 			)
 		)
-		(property "Value" "10"
+		(property "Value" "0"
 			(at 100.33 77.47 90)
 			(effects
