File: rvswdio-programmer/rvswdio-programmer.kicad_pcb (KiCad board)
At the start: 2 copper layers, 15.5 x 36.6 mm, 21 parts, among them J1 USB2.0-C_SMT, U1 CH32V003F4P6, U2 AMS1117, U3 CH217K

Commit message: spell misstake
Other:
- board text added: "RVSWDIO Programmer"
- board text removed: "RVSWDIO Programer"
Changed lines of the file:
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@@
 	(paper "A4")
 	(title_block
-		(title "RVSWDIO Programer")
-		(rev "1.0.0")
+		(title "RVSWDIO Programmer")
+		(rev "1.0.1")
 	)
 	(layers
@@
 		)
 	)
-	(gr_text "RVSWDIO Programer"
+	(gr_text "RVSWDIO Programmer"
 		(at 90.7 34.9 270)
 		(layer "F.SilkS")
@@
 			(justify left bottom)
 		)
-		(render_cache "RVSWDIO Programer" 270
+		(render_cache "RVSWDIO Programmer" 270
 			(polygon
 				(pts
@@
 			(polygon
 				(pts
-					(xy 91.556211 54.357555) (xy 91.646483 54.38019) (xy 91.729762 54.417421) (xy 91.805208 54.468488)
-					(xy 91.867892 54.530252) (xy 91.91894 54.603607) (xy 91.956144 54.685005) (xy 91.978789 54.773661)
-					(xy 91.986558 54.871175) (xy 91.978757 54.968608) (xy 91.956086 55.05655) (xy 91.91894 55.136692)
-					(xy 91.867938 55.208731) (xy 91.805271 55.269222) (xy 91.729762 55.319031) (xy 91.64652 55.354955)
-					(xy 91.554352 55.377046) (xy 91.451508 55.384684) (xy 91.39466 55.380751) (xy 91.39466 55.204396)
-					(xy 91.529898 55.204396) (xy 91.613351 55.185085) (xy 91.684081 55.149605) (xy 91.744465 55.09754)
-					(xy 91.790384 55.032619) (xy 91.818167 54.958084) (xy 91.827813 54.871175) (xy 91.818271 54.784196)
-					(xy 91.79081 54.709627) (xy 91.745491 54.644726) (xy 91.685626 54.592813) (xy 91.614619 54.557314)
-					(xy 91.529898 54.537955) (xy 91.529898 55.204396) (xy 91.39466 55.204396) (xy 91.39466 54.537955)
-					(xy 91.328348 54.552433) (xy 91.270305 54.577231) (xy 91.219186 54.612328) (xy 91.174109 54.658489)
-					(xy 91.128597 54.731057) (xy 91.100636 54.815312) (xy 91.090847 54.91426) (xy 91.099159 55.005296)
-					(xy 91.123002 55.084179) (xy 91.161785 55.153251) (xy 91.216339 55.214141) (xy 91.094779 55.318005)
-					(xy 91.044497 55.267465) (xy 91.00277 55.209284) (xy 90.969287 55.14259) (xy 90.945746 55.071528)
-					(xy 90.931216 54.993792) (xy 90.926203 54.908361) (xy 90.93408 54.800351) (xy 90.956846 54.703618)
-					(xy 90.993821 54.616345) (xy 91.045332 54.537298) (xy 91.108087 54.472083) (xy 91.183 54.419387)
-					(xy 91.266467 54.381099) (xy 91.357386 54.357797) (xy 91.457406 54.349802)
+					(xy 91.986558 55.738506) (xy 91.978764 55.835575) (xy 91.956681 55.918087) (xy 91.921411 55.988633)
+					(xy 91.872863 56.049159) (xy 91.812973 56.096975) (xy 91.738991 56.132617) (xy 91.647895 56.155526)
+					(xy 91.535796 56.163794) (xy 90.938 56.163794) (xy 90.938 55.975642) (xy 91.514254 55.975642) (xy 91.612561 55.96676)
+					(xy 91.686433 55.942795) (xy 91.741558 55.906057) (xy 91.782948 55.854962) (xy 91.80877 55.790045)
+					(xy 91.818068 55.707133) (xy 91.812031 55.636675) (xy 91.794854 55.576465) (xy 91.767219 55.524611)
+					(xy 91.728821 55.479743) (xy 91.68213 55.444478) (xy 91.625405 55.418254) (xy 91.556584 55.401477)
+					(xy 91.47305 55.395455) (xy 90.938 55.395455) (xy 90.938 55.207302) (xy 91.514254 55.207302) (xy 91.612561 55.19842)
+					(xy 91.686433 55.174455) (xy 91.741558 55.137718) (xy 91.782948 55.086623) (xy 91.80877 55.021706)
+					(xy 91.818068 54.938794) (xy 91.812031 54.868336) (xy 91.794854 54.808126) (xy 91.767219 54.756271)
+					(xy 91.728821 54.711404) (xy 91.682136 54.676178) (xy 91.625412 54.64998) (xy 91.55659 54.633218)
+					(xy 91.47305 54.627201) (xy 90.938 54.627201) (xy 90.938 54.438963) (xy 91.976813 54.438963) (xy 91.976813 54.619337)
+					(xy 91.822 54.619337) (xy 91.871221 54.661053) (xy 91.911861 54.710407) (xy 91.944414 54.768251)
+					(xy 91.967395 54.830976) (xy 91.981625 54.900524) (xy 91.986558 54.978032) (xy 91.980844 55.057809)
+					(xy 91.964342 55.129202) (xy 91.937576 55.193539) (xy 91.899834 55.251589) (xy 91.852481 55.299647)
+					(xy 91.794559 55.338607) (xy 91.849731 55.382412) (xy 91.896612 55.436554) (xy 91.935609 55.502311)
+					(xy 91.963513 55.573835) (xy 91.980652 55.652157)
 				)
 			)
 			(polygon
 				(pts
-					(xy 91.802338 55.825701) (xy 91.8575 55.863438) (xy 91.90298 55.911359) (xy 91.939542 55.970683)
-					(xy 91.964812 56.036366) (xy 91.980861 56.113431) (xy 91.986558 56.203972) (xy 91.804304 56.203972)
-					(xy 91.806271 56.160887) (xy 91.800016 56.085267) (xy 91.782326 56.021373) (xy 91.754081 55.967064)
-					(xy 91.715144 55.92076) (xy 91.667339 55.88417) (xy 91.609568 55.857055) (xy 91.539801 55.83976)
-					(xy 91.45544 55.833565) (xy 90.938 55.833565) (xy 90.938 55.645327) (xy 91.976813 55.645327) (xy 91.976813 55.825701)
+					(xy 91.556211 56.428343) (xy 91.646483 56.450978) (xy 91.729762 56.48821) (xy 91.805208 56.539277)
+					(xy 91.867892 56.601041) (xy 91.91894 56.674396) (xy 91.956144 56.755793) (xy 91.978789 56.844449)
+					(xy 91.986558 56.941964) (xy 91.978757 57.039397) (xy 91.956086 57.127338) (xy 91.91894 57.20748)
+					(xy 91.867938 57.279519) (xy 91.805271 57.340011) (xy 91.729762 57.38982) (xy 91.64652 57.425744)
+					(xy 91.554352 57.447834) (xy 91.451508 57.455472) (xy 91.39466 57.45154) (xy 91.39466 57.275184)
+					(xy 91.529898 57.275184) (xy 91.613351 57.255873) (xy 91.684081 57.220394) (xy 91.744465 57.168328)
+					(xy 91.790384 57.103407) (xy 91.818167 57.028872) (xy 91.827813 56.941964) (xy 91.818271 56.854985)
+					(xy 91.79081 56.780416) (xy 91.745491 56.715514) (xy 91.685626 56.663601) (xy 91.614619 56.628102)
+					(xy 91.529898 56.608743) (xy 91.529898 57.275184) (xy 91.39466 57.275184) (xy 91.39466 56.608743)
+					(xy 91.328348 56.623221) (xy 91.270305 56.648019) (xy 91.219186 56.683116) (xy 91.174109 56.729277)
+					(xy 91.128597 56.801845) (xy 91.100636 56.8861) (xy 91.090847 56.985048) (xy 91.099159 57.076085)
+					(xy 91.123002 57.154967) (xy 91.161785 57.224039) (xy 91.216339 57.28493) (xy 91.094779 57.388794)
+					(xy 91.044497 57.338253) (xy 91.00277 57.280072) (xy 90.969287 57.213379) (xy 90.945746 57.142317)
+					(xy 90.931216 57.064581) (xy 90.926203 56.97915) (xy 90.93408 56.871139) (xy 90.956846 56.774406)
+					(xy 90.993821 56.687133) (xy 91.045332 56.608086) (xy 91.108087 56.542872) (xy 91.183 56.490176)
+					(xy 91.266467 56.451887) (xy 91.357386 56.428585) (xy 91.457406 56.420591)
+				)
+			)
+			(polygon
+				(pts
+					(xy 91.802338 57.896489) (xy 91.8575 57.934227) (xy 91.90298 57.982148) (xy 91.939542 58.041472)
+					(xy 91.964812 58.107155) (xy 91.980861 58.184219) (xy 91.986558 58.27476) (xy 91.804304 58.27476)
+					(xy 91.806271 58.231676) (xy 91.800016 58.156056) (xy 91.782326 58.092162) (xy 91.754081 58.037852)
+					(xy 91.715144 57.991549) (xy 91.667339 57.954958) (xy 91.609568 57.927843) (xy 91.539801 57.910548)
+					(xy 91.45544 57.904354) (xy 90.938 57.904354) (xy 90.938 57.716116) (xy 91.976813 57.716116) (xy 91.976813 57.896489)
 				)
 			)
@@
 			(justify left bottom mirror)
 		)
-		(render_cache "74TH-G066-1.0.0" 90
+		(render_cache "74TH-G066-1.0.1" 90
 			(polygon
 				(pts
@@
 			(polygon
 				(pts
-					(xy 102.419626 55.772191) (xy 102.544161 55.796866) (xy 102.652373 55.835989) (xy 102.75218 55.891919)
-					(xy 102.831986 55.958125) (xy 102.894381 56.034912) (xy 102.94031 56.122412) (xy 102.968112 56.218091)
-					(xy 102.977643 56.324023) (xy 102.96815 56.428647) (xy 102.940385 56.523696) (xy 102.894381 56.611167)
-					(xy 102.831986 56.687954) (xy 102.75218 56.75416) (xy 102.652373 56.81009) (xy 102.544161 56.849213)
-					(xy 102.419626 56.873887) (xy 102.275982 56.882581) (xy 102.132338 56.873886) (xy 102.007834 56.84921)
-					(xy 101.899677 56.81009) (xy 101.79987 56.75416) (xy 101.720064 56.687954) (xy 101.657669 56.611167)
-					(xy 101.611616 56.523691) (xy 101.583824 56.428643) (xy 101.574322 56.324023) (xy 101.748796 56.324023)
-					(xy 101.757429 56.403029) (xy 101.782445 56.47194) (xy 101.823973 56.533037) (xy 101.884034 56.587658)
-					(xy 101.952888 56.62806) (xy 102.038705 56.659038) (xy 102.145017 56.67929) (xy 102.275982 56.68665)
-					(xy 102.406996 56.679289) (xy 102.513335 56.659035) (xy 102.599163 56.628057) (xy 102.668017 56.587658)
-					(xy 102.728077 56.533037) (xy 102.769605 56.47194) (xy 102.794621 56.403029) (xy 102.803254 56.324023)
-					(xy 102.794581 56.243972) (xy 102.769498 56.174422) (xy 102.727958 56.113032) (xy 102.668017 56.058421)
-					(xy 102.599163 56.018021) (xy 102.513335 55.987044) (xy 102.406996 55.96679) (xy 102.275982 55.959429)
-					(xy 102.145017 55.966789) (xy 102.038705 55.987041) (xy 101.952888 56.018019) (xy 101.884034 56.058421)
-					(xy 101.824092 56.113032) (xy 101.782552 56.174422) (xy 101.75747 56.243972) (xy 101.748796 56.324023)
-					(xy 101.574322 56.324023) (xy 101.583862 56.218095) (xy 101.611691 56.122417) (xy 101.657669 56.034912)
-					(xy 101.720064 55.958125) (xy 101.79987 55.891919) (xy 101.899677 55.835989) (xy 102.007834 55.796869)
-					(xy 102.132338 55.772193) (xy 102.275982 55.763497)
+					(xy 101.589965 56.18605) (xy 102.962 56.18605) (xy 102.962 55.991999) (xy 101.760508 55.991999)
+					(xy 101.760508 55.682287) (xy 101.589965 55.682287)
 				)
 			)
