File: rvswdio-programmer/rvswdio-programmer.kicad_sch (KiCad schematic)
At the start: 21 parts, among them J1 USB2.0-C_SMT, U1 CH32V003F4P6, U2 AMS1117, U3 CH217K

Commit message: spell misstake
Other:
- note added: "Interface Pins"
- note added: "Power"
- note added: "Programmer MCU"
- note added: "Programmer MCU SWDIO"
- note added: "Programmer USB"
- note added: "Target Connection"
- note added: "Target Power Switch"
- title: RVSWDIO Programer -> RVSWDIO Programmer
- moved on the sheet: C1, C2, C3, C4, C5, CH1, CH2, J1, R1, R10, R2, R3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
